Commit message: fixed gazebo sim issues

File: catkin_ws/src/haas_vf2/urdf/haas_vf2.urdf (robot description, URDF)
Before this commit: robot haas_vf2, 4 links, 3 joints
Links:
- removed link vf2_base_link
- added link world
- link base_link: mass None -> 30; geometry collision mesh filename=package://haas_vf2/meshes/Body2.stl; visual mesh filename=package://haas_vf2/meshes/Body2.stl
Joints:
- removed joint base_to_vf2
- added joint fixed_base_joint: type fixed, parent world, child base_link
- joint base_to_y_axis: parent vf2_base_link -> base_link

Commit message: now with spindle and part

File: catkin_ws/src/haas_vf2/urdf/haas_vf2.urdf (robot description, URDF)
Before this commit: robot haas_vf2, 4 links, 3 joints
Links:
- added link part, mass 1; collision mesh filename=package://haas_vf2/meshes/cube_body.stl; visual mesh filename=package://haas_vf2/meshes/cube_body.stl
- added link spindle, mass 1; collision mesh filename=package://haas_vf2/meshes/cylinder_body.stl; visual mesh filename=package://haas_vf2/meshes/cylinder_body.stl
Joints:
- added joint base_spindle_joint: type fixed, parent base_link, child spindle
- added joint fixed_part_joint: type fixed, parent x_axis_table, child part
